Commit message: Fix launch files to run gazebo world

File: urdf/my_bot.xacro (robot description, xacro)
@@ -1,34 +1,34 @@
 <?xml version='1.0'?>
 <robot name="my_bot" xmlns:xacro="http://www.ros.org/wiki/xacro">
-  <xacro:include filename="$(find rtab_bot)/urdf/my_bot.gazebo" />
-  <link name="robot_footprint"></link>
-  <joint name="robot_footprint_joint" type="fixed">
-    <origin xyz="0 0 0" rpy="0 0 0" />
-    <parent link="robot_footprint"/>
-    <child link="chassis" />
-  </joint>
-  <link name='chassis'>
-    <pose>0 0 0.071 0 0 0</pose>
-    <inertial>
-      <mass value="10.0"/>
-      <origin xyz="0 0 0" rpy="0 0 0"/>
-      <inertia
-          ixx="0.10833" ixy="0" ixz="0"
-          iyy="0.10833" iyz="0"
-          izz="0.2"
-      />
-    </inertial>
-    <collision name='collision'>
-      <origin xyz="0 0 0" rpy="0 0 0"/>
-      <geometry>
-        <cylinder radius="0.2" length="0.1"/>
-      </geometry>
-    </collision>
-    <visual name='chassis_visual'>
-      <origin xyz="0 0 0" rpy="0 0 0"/>
-      <geometry>
-        <cylinder radius="0.2" length="0.1"/>
-      </geometry>
-    </visual>
+    <xacro:include filename="$(find slam_project)/urdf/my_bot.gazebo" />
+    <link name="robot_footprint"></link>
+    <joint name="robot_footprint_joint" type="fixed">
+        <origin xyz="0 0 0" rpy="0 0 0" />
+        <parent link="robot_footprint"/>
+        <child link="chassis" />
+    </joint>
+    <link name='chassis'>
+        <pose>0 0 0.071 0 0 0</pose>
+        <inertial>
+            <mass value="10.0"/>
+            <origin xyz="0 0 0" rpy="0 0 0"/>
+            <inertia
+                ixx="0.10833" ixy="0" ixz="0"
+                iyy="0.10833" iyz="0"
+                izz="0.2"
+            />
+        </inertial>
+        <collision name='collision'>
+            <origin xyz="0 0 0" rpy="0 0 0"/>
+            <geometry>
+                <cylinder radius="0.2" length="0.1"/>
+            </geometry>
+        </collision>
+        <visual name='chassis_visual'>
+            <origin xyz="0 0 0" rpy="0 0 0"/>
+            <geometry>
+                <cylinder radius="0.2" length="0.1"/>
+            </geometry>
+        </visual>
   </link>
   <link name='caster'>

Commit message: Fix launching parameters for most scripts

File: urdf/my_bot.xacro (robot description, xacro)
@@ -151,5 +151,5 @@
   </link>
   <joint type="fixed" name="camera_joint">
-    <origin xyz="0.20 0 0" rpy="0 0 0"/>
+    <origin xyz="0.2 0.0 0.0" rpy="0 0 0"/>
     <child link="camera"/>
     <parent link="chassis"/>

Commit message: Restore RTAB MAP package

File: urdf/my_bot.xacro (robot description, xacro)
@@ -126,5 +126,5 @@
     <dynamics damping="0.1" friction="0.1"/>
   </joint>
-  <link name='camera'>
+  <link name='camera_depth_frame'>
     <pose>0 0 0 0 0 0</pose>
     <inertial>
@@ -152,5 +152,5 @@
   <joint type="fixed" name="camera_joint">
     <origin xyz="0.2 0.0 0.0" rpy="0 0 0"/>
-    <child link="camera"/>
+    <child link="camera_depth_frame"/>
     <parent link="chassis"/>
   </joint>

Commit message: Map the kitchen

File: urdf/my_bot.xacro (robot description, xacro)
@@ -155,3 +155,10 @@
     <parent link="chassis"/>
   </joint>
+  <link name='camera_optical_link'>
+  </link>
+  <joint type="fixed" name="camera_optical_joint">
+    <origin xyz="0.2 0.0 0.0" rpy="${-pi/2} 0 ${-pi/2}"/>
+    <child link="camera_optical_link"/>
+    <parent link="chassis"/>
+  </joint>
 </robot>

Commit message: Restore laser sensor

File: urdf/my_bot.xacro (robot description, xacro)
@@ -162,3 +162,32 @@
     <parent link="chassis"/>
   </joint>
+  <link name='hokuyo'>
+    <pose>0 0 0 0 0 0</pose>
+    <inertial>
+      <mass value="1.0"/>
+      <origin xyz="0 0 0" rpy="0 0 0"/>
+      <inertia
+          ixx="0.001667" ixy="0" ixz="0"
+          iyy="0.001667" iyz="0"
+          izz="0.001667"
+      />
+    </inertial>
+    <collision name='collision'>
+      <origin xyz="0 0 0" rpy="0 0 0"/>
+      <geometry>
+        <box size="0.1 0.1 0.1"/>
+      </geometry>
+    </collision>
+    <visual name='hokuyo_visual'>
+      <origin xyz="0 0 0" rpy="0 0 0"/>
+      <geometry>
+        <mesh filename="package://slam_project/meshes/hokuyo.dae"/>
+      </geometry>
+    </visual>
+  </link>
+  <joint type="fixed" name="hokuyo_joint">
+    <origin xyz="0 0 0.08" rpy="0 0 0"/>
+    <child link="hokuyo"/>
+    <parent link="chassis"/>
+  </joint>
 </robot>
